Commit message: add gazebo sim

File: my_model/urdf/my_robot.xacro (robot description, xacro)
@@ -12,4 +12,5 @@
             <parent link="${parent}"/>
             <child link="wheel_${number}" />
+            <axis xyz="0 1 0"/>
         </joint>
         <link name="wheel_${number}">
@@ -36,4 +37,15 @@
             </collision>
         </link>
+        <gazebo reference="wheel_${number}">
+            <material>Gazebo/Gray</material>
+        </gazebo>
+        <transmission name="simple_trans_${number}">
+            <type>transmission_interface/SimpleTransmission</type>
+            <joint name="base_to_wheel_joint_${number}" />
+            <actuator name="actuator_${number}">
+                <mechanicalReduction>1</mechanicalReduction>
+                <hardwareInterface>VelocityJointInterface</hardwareInterface>
+            </actuator>
+        </transmission>
     </xacro:macro>
     <xacro:macro name="my_robot">
@@ -61,8 +73,11 @@
             </collision>
         </link>
-        <base_to_wheel_joint parent="base_link" number="front_left" x_loc="${base_l/2}" y_loc="${base_w/2 + wheel_l/2}+" z_loc="-${base_h/2}"/>
-        <base_to_wheel_joint parent="base_link" number="front_righ" x_loc="${base_l/2}" y_loc="-${base_w/2 + wheel_l/2}+" z_loc="-${base_h/2}"/>
-        <base_to_wheel_joint parent="base_link" number="back_left" x_loc="-${base_l/2}" y_loc="${base_w/2 + wheel_l/2}+" z_loc="-${base_h/2}"/>
-        <base_to_wheel_joint parent="base_link" number="back_righ" x_loc="-${base_l/2}" y_loc="-${base_w/2 + wheel_l/2}+" z_loc="-${base_h/2}"/>
+        <gazebo reference="base_link">
+            <material>Gazebo/Yellow</material>
+        </gazebo>
+        <base_to_wheel_joint parent="base_link" number="front_left" x_loc="${base_l/2}" y_loc="${base_w/2 + wheel_l/2}" z_loc="${-base_h/2}"/>
+        <base_to_wheel_joint parent="base_link" number="front_righ" x_loc="${base_l/2}" y_loc="${-base_w/2 - wheel_l/2}" z_loc="${-base_h/2}"/>
+        <base_to_wheel_joint parent="base_link" number="back_left" x_loc="${-base_l/2}" y_loc="${base_w/2 + wheel_l/2}" z_loc="${-base_h/2}"/>
+        <base_to_wheel_joint parent="base_link" number="back_righ" x_loc="${-base_l/2}" y_loc="${-base_w/2 - wheel_l/2}" z_loc="${-base_h/2}"/>
     </xacro:macro>
 </robot>

File: my_model/urdf/my_robot_with_rplidar.xacro (robot description, xacro)
@@ -1,5 +1,5 @@
 <?xml version="1.0"?>
 <robot name="deeptuuk" xmlns:xacro="http://www.ros.org/wiki/xacro">
-    <xacro:include filename="my_robot.urdf"/>
+    <xacro:include filename="my_robot.xacro"/>
     <xacro:include filename="rplidar.xacro" />
 	<xacro:property name="rplidar_offset_x" value="0" />
@@ -13,4 +13,26 @@
 		<child link="laser_link"/>
 	</joint>
-	<xacro:rplidar prefix="laser"/>
+	<rplidar/>
+	<gazebo>
+		<plugin name="skid_steer_drive_controller" filename="libgazebo_ros_skid_steer_drive.so">
+			<updateRate>100.0</updateRate>
+			<alwaysOn>true</alwaysOn>
+			<covariance_x>0.0001</covariance_x>
+			<covariance_y>0.0001</covariance_y>
+			<covariance_yaw>0.01</covariance_yaw>
+			<robotNamespace>/</robotNamespace>
+			<leftFrontJoint>base_to_wheel_joint_front_left</leftFrontJoint>
+			<rightFrontJoint>base_to_wheel_joint_front_righ</rightFrontJoint>
+			<leftRearJoint>base_to_wheel_joint_back_left</leftRearJoint>
+			<rightRearJoint>base_to_wheel_joint_back_righ</rightRearJoint>
+			<wheelSeparation>0.24</wheelSeparation>
+			<wheelDiameter>0.08</wheelDiameter>
+			<robotBaseFrame>base_link</robotBaseFrame>
+			<torque>50</torque>
+			<commandTopic>cmd_vel</commandTopic>
+			<odometryTopic>odom</odometryTopic>
+			<odometryFrame>odom</odometryFrame>
+			<broadcastTF>true</broadcastTF>
+		</plugin>
+	</gazebo>
 </robot>

File: my_model/urdf/rplidar.xacro (robot description, xacro)
@@ -1,6 +1,6 @@
 <?xml version="1.0"?>
 <robot xmlns:xacro="http://www.ros.org/wiki/xacro" name="laser">
-	<xacro:macro name="rplidar" params="prefix:=laser">
-		<link name="${prefix}_link">
+	<xacro:macro name="rplidar">
+		<link name="laser_link">
 			<inertial>
 				<mass value="0.1" />
@@ -24,4 +24,7 @@
 			</collision>
 		</link>
+		<gazebo reference="laser_link">
+			<material>Gazebo/Black</material>
+		</gazebo>
 	</xacro:macro>
 </robot>
