Commit message: add pi_model

File: my_model/urdf/my_pi.xacro (robot description, xacro)
@@ -2,9 +2,9 @@
 <robot xmlns:xacro="http://www.ros.org/wiki/xacro">
     <xacro:property name="PI" value="3.14159"/>
-    <xacro:property name="base_l" value="0.3"/>
-    <xacro:property name="base_w" value="0.2"/>
-    <xacro:property name="base_h" value="0.1"/>
+    <xacro:property name="base_l" value="0.1"/>
+    <xacro:property name="base_r" value="0.15"/>
     <xacro:property name="wheel_l" value="0.04"/>
     <xacro:property name="wheel_r" value="0.04"/>
+    <xacro:property name="fix_r" value="0.02"/>
     <xacro:macro name="base_to_wheel_joint" params="parent number x_loc y_loc z_loc">
         <joint name="base_to_wheel_joint_${number}" type="continuous">
@@ -46,8 +46,43 @@
             <joint name="base_to_wheel_joint_${number}" />
             <actuator name="actuator_${number}">
-                <mechanicalReduction>100</mechanicalReduction>
+                <mechanicalReduction>1</mechanicalReduction>
                 <hardwareInterface>VelocityJointInterface</hardwareInterface>
             </actuator>
         </transmission>
+    </xacro:macro>
+    <xacro:macro name="base_to_fix_joint" params="parent number x_loc y_loc z_loc">
+        <joint name="base_to_wheel_fix_${number}" type="fixed">
+            <origin xyz="${x_loc} ${y_loc} ${z_loc}" rpy="0 0 0" />
+            <parent link="${parent}"/>
+            <child link="fix_${number}" />
+        </joint>
+        <link name="fix_${number}">
+            <visual>
+                <origin xyz=" 0 0 0" rpy="0 0 0" />
+                <geometry>
+                    <sphere radius="${fix_r}"/>
+                </geometry>
+                <material name="gray">
+                    <color rgba="0.75 0.75 0.75 1"/>
+                </material>
+            </visual>
+            <inertial>
+                <mass value="1" />
+                <origin xyz="0 0 0" />
+                <inertia ixx="0.00053" ixy="0.00000" ixz="0.00000"
+                        iyy="0.00053" iyz="0.00000" izz="0.00080" />
+            </inertial>
+            <collision>
+                <origin xyz="0 0 0" rpy="0 0 0" />
+                <geometry>
+                    <sphere radius="${fix_r}"/>
+                </geometry>
+            </collision>
+        </link>
+        <gazebo reference="fix_${number}">
+            <material>Gazebo/Gray</material>
+            <mu1>0.0</mu1>
+            <mu2>0.0</mu2>
+        </gazebo>
     </xacro:macro>
     <xacro:macro name="my_robot">
@@ -56,5 +91,5 @@
                 <origin xyz=" 0 0 0" rpy="0 0 0" />
                 <geometry>
-                    <box size="${base_l} ${base_w} ${base_h}" />
+                    <cylinder radius="${base_r}" length = "${base_l}"/>
                 </geometry>
                 <material name="yellow">
@@ -71,5 +106,5 @@
                 <origin xyz="0 0 0" rpy="0 0 0" />
                 <geometry>
-                    <box size="${base_l} ${base_w} ${base_h}" />
+                    <cylinder radius="${base_r}" length = "${base_l}"/>
                 </geometry>
             </collision>
@@ -78,8 +113,8 @@
             <material>Gazebo/Yellow</material>
         </gazebo>
-        <base_to_wheel_joint parent="base_link" number="front_left" x_loc="${base_l/2}" y_loc="${base_w/2 + wheel_l/2}" z_loc="${-base_h/2}"/>
-        <base_to_wheel_joint parent="base_link" number="front_righ" x_loc="${base_l/2}" y_loc="${-base_w/2 - wheel_l/2}" z_loc="${-base_h/2}"/>
-        <base_to_wheel_joint parent="base_link" number="back_left" x_loc="${-base_l/2}" y_loc="${base_w/2 + wheel_l/2}" z_loc="${-base_h/2}"/>
-        <base_to_wheel_joint parent="base_link" number="back_righ" x_loc="${-base_l/2}" y_loc="${-base_w/2 - wheel_l/2}" z_loc="${-base_h/2}"/>
+        <base_to_wheel_joint parent="base_link" number="left" x_loc="0" y_loc="${base_r + wheel_l/2}" z_loc="${-base_l/2}"/>
+        <base_to_wheel_joint parent="base_link" number="righ" x_loc="0" y_loc="${-base_r - wheel_l/2}" z_loc="${-base_l/2}"/>
+        <base_to_fix_joint parent="base_link" number="front" x_loc="${base_r}" y_loc="0" z_loc="${-base_l/2 - fix_r}"/>
+        <base_to_fix_joint parent="base_link" number="back" x_loc="${-base_r}" y_loc="0" z_loc="${-base_l/2 - fix_r}"/>
     </xacro:macro>
 </robot>

File: my_model/urdf/my_robot_2.xacro (robot description, xacro)
@@ -39,6 +39,4 @@
         <gazebo reference="wheel_${number}">
             <material>Gazebo/Gray</material>
-            <mu1>100</mu1>
-            <mu2>100</mu2>
         </gazebo>
         <transmission name="simple_trans_${number}">
@@ -46,5 +44,5 @@
             <joint name="base_to_wheel_joint_${number}" />
             <actuator name="actuator_${number}">
-                <mechanicalReduction>100</mechanicalReduction>
+                <mechanicalReduction>1</mechanicalReduction>
                 <hardwareInterface>VelocityJointInterface</hardwareInterface>
             </actuator>
@@ -56,5 +54,5 @@
                 <origin xyz=" 0 0 0" rpy="0 0 0" />
                 <geometry>
-                    <box size="${base_l} ${base_w} ${base_h}" />
+                    <box size="0.15 0.1 0.05" />
                 </geometry>
                 <material name="yellow">
@@ -71,5 +69,5 @@
                 <origin xyz="0 0 0" rpy="0 0 0" />
                 <geometry>
-                    <box size="${base_l} ${base_w} ${base_h}" />
+                    <box size="0.15 0.1 0.05" />
                 </geometry>
             </collision>

File: my_model/urdf/my_robot_with_rplidar_2.xacro (robot description, xacro)
@@ -1,5 +1,5 @@
 <?xml version="1.0"?>
 <robot name="deeptuuk" xmlns:xacro="http://www.ros.org/wiki/xacro">
-    <xacro:include filename="my_robot.xacro"/>
+    <xacro:include filename="my_robot_2.xacro"/>
     <xacro:include filename="rplidar.xacro" />
 	<xacro:property name="rplidar_offset_x" value="0" />
@@ -29,5 +29,5 @@
 			<wheelDiameter>0.08</wheelDiameter>
 			<robotBaseFrame>base_link</robotBaseFrame>
-			<torque>100</torque>
+			<torque>5000</torque>
 			<commandTopic>cmd_vel</commandTopic>
 			<odometryTopic>odom</odometryTopic>
